File: pcb/esp8266-incubator.brd (EAGLE design)
At the start: 48.3 x 91.7 mm, 48 parts, among them Q1 MOSFET-PGDS_TO220V

Commit message: Renamed source files.
Parts:
- C4: value 100nF -> 1000nF
- D3: value (none) -> 1N4007
- R12, R13, R14, R15: value 12K -> 10K
- R17: value 12K -> 100R
- R18: value 12K -> 120K
- moved RIN 0.25 mm to (33.8, 3.30)
- moved ROUT2 0.25 mm to (44.7, 43.9)
Changed lines of the file:
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@@
 <attribute name="VALUE" x="20.701" y="35.941" size="1.27" layer="28" rot="MR90"/>
 </element>
-<element name="RIN" library="SparkFun-Connectors" package="SCREWTERMINAL-5MM-2" value="" x="33.782" y="3.556" smashed="yes">
-<attribute name="NAME" x="30.146" y="2.08" size="1.27" layer="25" font="vector" ratio="15" rot="R90"/>
-<attribute name="STOREFRONT_ID" value="PRT-08432" x="33.782" y="3.556" size="1.778" layer="27" display="off"/>
+<element name="RIN" library="SparkFun-Connectors" package="SCREWTERMINAL-5MM-2" value="" x="33.782" y="3.302" smashed="yes">
+<attribute name="NAME" x="30.146" y="1.826" size="1.27" layer="25" font="vector" ratio="15" rot="R90"/>
+<attribute name="STOREFRONT_ID" value="PRT-08432" x="33.782" y="3.302" size="1.778" layer="27" display="off"/>
 </element>
 <element name="ROUT1" library="SparkFun-Connectors" package="SCREWTERMINAL-5MM-2" value="" x="44.704" y="56.134" smashed="yes" rot="R90">
@@
 <attribute name="VALUE" x="24.257" y="2.159" size="1.27" layer="28" ratio="10" rot="MR0"/>
 </element>
-<element name="R12" library="rcl" package="R0805" value="12K" x="19.304" y="14.732" smashed="yes" rot="MR90">
+<element name="R12" library="rcl" package="R0805" value="10K" x="19.304" y="14.732" smashed="yes" rot="MR90">
 <attribute name="NAME" x="18.288" y="16.637" size="1.27" layer="26" font="vector" ratio="15" rot="MR270"/>
 <attribute name="VALUE" x="16.764" y="14.097" size="1.27" layer="28" rot="MR90"/>
@@
 <attribute name="VALUE" x="19.431" y="12.319" size="1.27" layer="28" rot="MR90"/>
 </element>
-<element name="R13" library="rcl" package="R0805" value="12K" x="21.336" y="11.43" smashed="yes" rot="MR180">
+<element name="R13" library="rcl" package="R0805" value="10K" x="21.336" y="11.43" smashed="yes" rot="MR180">
 <attribute name="NAME" x="19.431" y="10.922" size="1.27" layer="26" font="vector" ratio="15" rot="MR0"/>
 <attribute name="VALUE" x="20.701" y="13.97" size="1.27" layer="28" rot="MR180"/>
 </element>
-<element name="R14" library="rcl" package="R0805" value="12K" x="20.066" y="36.83" smashed="yes" rot="MR0">
+<element name="R14" library="rcl" package="R0805" value="10K" x="20.066" y="36.83" smashed="yes" rot="MR0">
 <attribute name="NAME" x="14.351" y="37.338" size="1.27" layer="26" font="vector" ratio="15" rot="MR180"/>
 <attribute name="VALUE" x="20.701" y="34.29" size="1.27" layer="28" rot="MR0"/>
@@
 <attribute name="VALUE" x="19.431" y="6.477" size="1.27" layer="28" rot="MR90"/>
 </element>
-<element name="R15" library="rcl" package="R0805" value="12K" x="19.304" y="8.382" smashed="yes" rot="MR270">
+<element name="R15" library="rcl" package="R0805" value="10K" x="19.304" y="8.382" smashed="yes" rot="MR270">
 <attribute name="NAME" x="18.288" y="10.287" size="1.27" layer="26" font="vector" ratio="15" rot="MR270"/>
 <attribute name="VALUE" x="21.844" y="9.017" size="1.27" layer="28" rot="MR270"/>
 </element>
-<element name="ROUT2" library="SparkFun-Connectors" package="SCREWTERMINAL-5MM-2" value="" x="44.704" y="43.688" smashed="yes" rot="R90">
-<attribute name="NAME" x="40.052" y="43.736" size="1.27" layer="25" font="vector" ratio="15" rot="R90"/>
-<attribute name="STOREFRONT_ID" value="PRT-08432" x="44.704" y="43.688" size="1.778" layer="27" rot="R90" display="off"/>
+<element name="ROUT2" library="SparkFun-Connectors" package="SCREWTERMINAL-5MM-2" value="" x="44.704" y="43.942" smashed="yes" rot="R90">
+<attribute name="NAME" x="40.052" y="43.99" size="1.27" layer="25" font="vector" ratio="15" rot="R90"/>
+<attribute name="STOREFRONT_ID" value="PRT-08432" x="44.704" y="43.942" size="1.778" layer="27" rot="R90" display="off"/>
 </element>
 <element name="ALARM" library="SparkFun" package="BUZZER-12MM" value="BUZZERPTH" x="8.636" y="72.898" smashed="yes">
@@
 <attribute name="VALUE" x="14.478" y="63.246" size="1.27" layer="27" ratio="10" rot="R270"/>
 </element>
-<element name="R17" library="rcl" package="R0805" value="12K" x="23.114" y="61.722" smashed="yes" rot="MR90">
+<element name="R17" library="rcl" package="R0805" value="100R" x="23.114" y="61.722" smashed="yes" rot="MR90">
 <attribute name="NAME" x="23.876" y="59.563" size="1.27" layer="26" font="vector" ratio="15" rot="MR270"/>
 <attribute name="VALUE" x="20.574" y="61.087" size="1.27" layer="28" rot="MR90"/>
 </element>
-<element name="R18" library="rcl" package="R0805" value="12K" x="25.146" y="61.722" smashed="yes" rot="MR90">
+<element name="R18" library="rcl" package="R0805" value="120K" x="25.146" y="61.722" smashed="yes" rot="MR90">
 <attribute name="NAME" x="25.908" y="59.563" size="1.27" layer="26" font="vector" ratio="15" rot="MR270"/>
 <attribute name="VALUE" x="22.606" y="61.087" size="1.27" layer="28" rot="MR90"/>
 </element>
-<element name="D3" library="diode" package="MELF-MLL41" value="" x="9.398" y="43.688" smashed="yes" rot="MR90">
+<element name="D3" library="diode" package="MELF-MLL41" value="1N4007" x="9.398" y="43.688" smashed="yes" rot="MR90">
 <attribute name="NAME" x="11.303" y="42.672" size="1.27" layer="26" font="vector" ratio="15" rot="MR90"/>
 <attribute name="VALUE" x="7.112" y="41.148" size="0.4064" layer="28" font="vector" rot="MR90"/>
 </element>
-<element name="C4" library="rcl" package="C0805" value="100nF" x="6.604" y="43.688" smashed="yes" rot="MR270">
+<element name="C4" library="rcl" package="C0805" value="1000nF" x="6.604" y="43.688" smashed="yes" rot="MR270">
 <attribute name="NAME" x="7.112" y="41.656" size="1.27" layer="26" font="vector" ratio="15" rot="MR270"/>
 <attribute name="VALUE" x="9.144" y="44.958" size="1.27" layer="28" rot="MR270"/>
@@
 <wire x1="44.704" y1="61.134" x2="42.338" y2="61.134" width="2.54" layer="1"/>
 <wire x1="42.338" y1="61.134" x2="41.148" y2="59.944" width="2.54" layer="1"/>
-<wire x1="41.148" y1="59.944" x2="41.148" y2="48.514" width="2.54" layer="1"/>
-<wire x1="41.148" y1="48.514" x2="41.148" y2="40.386" width="2.54" layer="1"/>
+<wire x1="41.148" y1="59.944" x2="41.148" y2="49.022" width="2.54" layer="1"/>
+<wire x1="41.148" y1="48.942" x2="41.148" y2="40.386" width="2.54" layer="1"/>
 <wire x1="41.148" y1="40.386" x2="32.512" y2="31.75" width="2.54" layer="1"/>
 <wire x1="32.512" y1="31.75" x2="28.384" y2="31.75" width="2.54" layer="1"/>
-<wire x1="44.704" y1="48.688" x2="41.322" y2="48.688" width="2.54" layer="1"/>
-<wire x1="41.322" y1="48.688" x2="41.148" y2="48.514" width="2.54" layer="1"/>
+<wire x1="44.704" y1="48.942" x2="41.148" y2="48.942" width="2.54" layer="1"/>
+<wire x1="41.148" y1="48.942" x2="41.148" y2="49.022" width="2.54" layer="1"/>
 </signal>
 <signal name="N$17">
@@
 <contactref element="ROUT1" pad="1"/>
 <contactref element="ROUT2" pad="1"/>
-<wire x1="33.782" y1="3.556" x2="33.782" y2="7.366" width="2.54" layer="16"/>
+<wire x1="33.782" y1="3.302" x2="33.782" y2="7.366" width="2.54" layer="16"/>
 <wire x1="33.782" y1="7.366" x2="35.052" y2="8.636" width="2.54" layer="16"/>
 <wire x1="35.052" y1="8.636" x2="35.052" y2="34.036" width="2.54" layer="16"/>
-<wire x1="35.052" y1="34.036" x2="44.704" y2="43.688" width="2.54" layer="16"/>
-<wire x1="44.704" y1="43.688" x2="42.672" y2="43.688" width="2.54" layer="16"/>
-<wire x1="42.672" y1="43.688" x2="41.148" y2="45.212" width="2.54" layer="16"/>
-<wire x1="44.704" y1="56.134" x2="42.926" y2="56.134" width="2.54" layer="16"/>
-<wire x1="42.926" y1="56.134" x2="41.148" y2="54.356" width="2.54" layer="16"/>
-<wire x1="41.148" y1="54.356" x2="41.148" y2="45.212" width="2.54" layer="16"/>
+<wire x1="35.052" y1="34.036" x2="44.704" y2="43.942" width="2.54" layer="16"/>
+<wire x1="44.704" y1="43.942" x2="42.926" y2="43.942" width="2.54" layer="16"/>
+<wire x1="42.926" y1="43.942" x2="41.148" y2="45.72" width="2.54" layer="16"/>
+<wire x1="41.148" y1="45.72" x2="41.148" y2="54.61" width="2.54" layer="16"/>
+<wire x1="44.704" y1="56.134" x2="42.672" y2="56.134" width="2.54" layer="16"/>
+<wire x1="42.672" y1="56.134" x2="41.148" y2="54.61" width="2.54" layer="16"/>
 </signal>
 <signal name="P230">
 <contactref element="RELAY_NC" pad="NC"/>
 <contactref element="RIN" pad="2"/>
-<wire x1="38.782" y1="3.556" x2="38.782" y2="17.692" width="2.54" layer="16"/>
+<wire x1="38.782" y1="3.302" x2="38.782" y2="17.692" width="2.54" layer="16"/>
 <wire x1="38.782" y1="17.692" x2="42.584" y2="21.494" width="2.54" layer="16"/>
 </signal>

Commit message: Designed new version schematics and board design.
Parts:
- removed ACT: RED, led:1206
- added ACT_LED, ALARM_LED, FAN_LED, PWR_LED, RELAY_LED: RED, led:1206
- added R19, R21: 10K, rcl:R0805
- added R20: 100R, rcl:R0805
- added R22: 1K, rcl:R0805
- added R23: 470R, rcl:R0805
- added R24, R25, R26, R27: 12K, rcl:R0805
- added RST: (no value), SparkFun-Retired:TACTILE-PTH
- added T7, T8: BSS138L, we-transistor:SOT23
- C1: value 220uF -> 1000nF; device rcl:E2,5-6 -> rcl:C0805
- C2: value 100nF -> 220uF; device rcl:C0805 -> rcl:E2,5-6
- C4: value 1000nF -> 100nF
- D1: value PMLL4150 -> 1N4007; device diode:SOD80C -> diode:MELF-MLL41
- D2: value PMLL4150 -> LL4148
- D3: value 1N4007 -> LL4148; device diode:MELF-MLL41 -> diode:SOD80C
- Q1: value MOSFET-PGDS_TO220V -> IRF9540N
- R1: value 82R -> 12K
- R10: value 12K -> 1K
- R11, R9: value 12K -> 100R
- R13, R15, R6: value 10K -> 100R
- R16: value 100 -> 1K
- R17: value 100R -> 82R
- R18: value 120K -> 10K
- R2: value 12K -> 82R
- R4: value 470R -> 12K
- R5: value 10K -> 470R
- R7, R8: value 12K -> 10K
- T3, T5, T6: value (none) -> BSS138L; device transistor:SOT23-BEC -> we-transistor:SOT23
- moved R11 57.6 mm to (19.3, 18.0), turned to 90 degrees
- moved R5 39.0 mm to (43.2, 75.7), flipped to the top
- moved C4 37.1 mm to (18.0, 79.0), turned to 180 degrees
- moved ALARM 35.3 mm to (32.0, 46.5)
- moved R1 26.8 mm to (37.6, 70.1), turned to 270 degrees
- moved R15 23.2 mm to (21.3, 31.5), turned to 180 degrees
- moved T3 21.0 mm to (19.6, 58.4), turned to 0 degrees
- moved C3 20.5 mm to (7.87, 61.2), turned to 0 degrees
- moved T6 20.3 mm to (21.8, 28.7), turned to 180 degrees
- moved R9 20.1 mm to (18.5, 54.9), turned to 90 degrees
- moved R4 19.7 mm to (24.1, 80.8), flipped to the bottom
- moved D3 19.6 mm to (24.9, 31.8)
- moved D1 18.4 mm to (9.40, 43.9), turned to 270 degrees
- moved R17 18.1 mm to (10.4, 74.7), turned to 270 degrees
- moved R18 17.5 mm to (7.87, 59.2), turned to 0 degrees
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- renumbered U$1 to U$1000, U$2 to PWR_SUPPLY
Connections:
- removed net FANOUT: C4.1, D3.A, FAN.1, Q1.3
- removed net N$3 (its old number): R2.1, T2.B
- new net N$16: D3.A, RELAY_NC.2, T7.3
- new net N$19: ALARM_LED.C, R22.1
- new net N$20: ALARM.-, R22.2, T8.3
- new net N$21: PWR_LED.C, R17.1
- new net N$22: FAN_LED.C, R10.1
- new net N$23: R6.1, T3.1
- new net N$24: R10.2, R8.2, R9.2, T3.3
- new net N$25: C1.2, D1.A, FAN.2, Q1.2
- new net N$26: R23.2, RST.1, RST.2
- new net N$7: R4.1, T2.B
- net +12V: now also Q1.3, R8.1; no longer C4.2, D3.C, FAN.2
- net +3V3: now also ACT_LED.A, ALARM.+, ALARM_LED.A, C3.2, D2.C, D3.C, FAN_LED.A, PWR_LED.A, R14.1, R18.2, R19.2, R24.2, R25.2, R26.2, R27.2, RELAY_LED.A, RELAY_NC.1; no longer ACT.A, C2.2, D1.C, R10.2, R11.2, R15.1, R5.2, R6.2, R8.2, R9.2, T6.E
- net BUZZER: now also R20.2, R21.1; no longer R16.2
- net DTR: now also R3.2, T2.E; no longer R2.2, T1.E
- net EN: now also R27.1; no longer R11.1
- net FAN: now also R6.2, R7.1; no longer R17.2, R18.2
- net GND: now also C1.1, C2.-, C4.1, D1.C, FAN.1, R1.2, R12.2, R17.2, R21.2, RST.3, RST.4, T3.2, T5.2, T6.2, T7.2, T8.2; no longer ALARM.-, C1.-, C2.1, D2.A, Q1.2, R18.1, RELAY_NC.2, T3.E, T5.E
- net GPIO0: now also R24.1, R5.1, T2.C; no longer R4.1, R8.1, T1.C
- net GPIO13: now also R18.1; no longer R5.1
- net GPIO14: now also R19.1; no longer R6.1
- net GPIO16: now also R2.2; no longer R1.2
- net GPIO2: now also R25.1; no longer R9.1
- net N$1: now also ACT_LED.C, R2.1; no longer ACT.C, R1.1
- net N$11: now also R11.1, T5.1; no longer R14.1, T3.B
- net N$12: now also R13.1, T6.1; no longer R12.1, T5.B
- net N$13: now also R14.2, R15.2, T6.3; no longer R13.2, T5.C
- net N$14: now also R15.1, T7.1; no longer R13.1, R15.2, T6.B
- net N$15: now also R16.1, RELAY_LED.C; no longer D2.C, RELAY_NC.1, T6.C
- net N$18: now also R9.1; no longer R17.1
- net N$2: now also C2.+; no longer C1.+
- net N$4: now also R5.2; no longer R4.2
- net N$5: now also R1.1; no longer R7.1
- net N$8: now also R20.1, T8.1; no longer ALARM.+, R16.1
- net N$9: now also D2.A, R16.2, T5.3; no longer D1.A, T3.C
- net NRST: now also C4.2, R23.1, R26.1, T1.C; no longer C3.2, R10.1, T2.C
- net P230: now also RELAY_NO.C; no longer RELAY_NC.NC
- net R230: now also RELAY_NC.NC; no longer RELAY_NO.C
- net RELAY: now also R11.2, R12.1, R13.2; no longer R12.2, R14.2
- net RST: now also R4.2, T1.E; no longer R3.2, T2.E
Routing:
- net N$9: track 8.56 -> 78.8 mm, vias 0 -> 1
- net N$20: track 0.00 -> 44.1 mm
- net +3V3: track 151.3 -> 189.1 mm, vias 2 -> 3
- net N$24: track 0.00 -> 25.1 mm
- net FANOUT: track 22.7 -> 0.00 mm
- net N$25: track 0.00 -> 19.1 mm
- net NRST: track 12.5 -> 30.4 mm
- net R230: track 43.5 -> 30.4 mm
- net N$17: track 18.4 -> 30.1 mm
- net N$16: track 0.00 -> 11.5 mm
- net N$26: track 0.00 -> 9.51 mm
- net N$21: track 0.00 -> 9.10 mm, vias 0 -> 1
- net N$8: track 11.3 -> 2.30 mm
- net N$14: track 9.84 -> 1.99 mm
- net N$2: track 16.2 -> 23.7 mm
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Other:
- board text added: "3V3"
- board text added: "ESP8266 INCUBATOR v0.1.1"
- board text added: "HIGH"
- board text added: "PWR_SUPPLY"
- board text removed: "ESP8266 INCUBATOR v0.1.0"
