File: pcb/esp8266-incubator.brd (EAGLE design)
At the start: 48.3 x 91.7 mm, 64 parts, among them Q1 IRF9540N, T3 BSS138L, T5 BSS138L, T6 BSS138L, T7 BSS138L, T8 BSS138L

Commit message: Design update.
Parts:
- T1, T2: value (none) -> S8050
Changed lines of the file:
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@@
 <attribute name="VALUE" x="14.097" y="72.136" size="1.27" layer="28" rot="MR180"/>
 </element>
-<element name="T2" library="transistor" package="SOT23-BEC" value="" x="28.194" y="81.788" smashed="yes" rot="MR90">
+<element name="T2" library="transistor" package="SOT23-BEC" value="S8050" x="28.194" y="81.788" smashed="yes" rot="MR90">
 <attribute name="NAME" x="29.337" y="83.693" size="1.27" layer="26" font="vector" ratio="15" rot="MR0"/>
 <attribute name="VALUE" x="25.019" y="79.883" size="1.27" layer="28" rot="MR90"/>
 </element>
-<element name="T1" library="transistor" package="SOT23-BEC" value="" x="20.066" y="81.788" smashed="yes" rot="MR270">
+<element name="T1" library="transistor" package="SOT23-BEC" value="S8050" x="20.066" y="81.788" smashed="yes" rot="MR270">
 <attribute name="NAME" x="21.209" y="83.693" size="1.27" layer="26" font="vector" ratio="15" rot="MR0"/>
 <attribute name="VALUE" x="23.241" y="83.693" size="1.27" layer="28" rot="MR270"/>

Commit message: Updated some resistor values.
Parts:
- R1, R24, R25, R26, R27, R3, R4: value 12K -> 10K
Changed lines of the file:
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@@
 <attribute name="VALUE" x="23.241" y="83.693" size="1.27" layer="28" rot="MR270"/>
 </element>
-<element name="R3" library="rcl" package="R0805" value="12K" x="24.13" y="82.804" smashed="yes" rot="MR180">
+<element name="R3" library="rcl" package="R0805" value="10K" x="24.13" y="82.804" smashed="yes" rot="MR180">
 <attribute name="NAME" x="25.019" y="83.82" size="1.27" layer="26" font="vector" ratio="15" rot="MR0"/>
 <attribute name="VALUE" x="23.495" y="85.344" size="1.27" layer="28" rot="MR180"/>
 </element>
-<element name="R4" library="rcl" package="R0805" value="12K" x="24.13" y="80.772" smashed="yes" rot="MR0">
+<element name="R4" library="rcl" package="R0805" value="10K" x="24.13" y="80.772" smashed="yes" rot="MR0">
 <attribute name="NAME" x="22.987" y="79.756" size="1.27" layer="26" font="vector" ratio="15" rot="MR180"/>
 <attribute name="VALUE" x="24.765" y="78.232" size="1.27" layer="28" rot="MR0"/>
@@
 <attribute name="VALUE" x="18.796" y="19.939" size="1.27" layer="27" ratio="10"/>
 </element>
-<element name="R1" library="rcl" package="R0805" value="12K" x="37.592" y="70.104" smashed="yes" rot="R270">
+<element name="R1" library="rcl" package="R0805" value="10K" x="37.592" y="70.104" smashed="yes" rot="R270">
 <attribute name="NAME" x="36.449" y="66.548" size="1.27" layer="25" font="vector" ratio="15"/>
 <attribute name="VALUE" x="35.052" y="70.739" size="1.27" layer="27" rot="R270"/>
@@
 <attribute name="NAME" x="40.386" y="78.74" size="1.27" layer="25" font="vector" ratio="15" rot="R90"/>
 </element>
-<element name="R24" library="rcl" package="R0805" value="12K" x="28.448" y="70.358" smashed="yes" rot="MR0">
+<element name="R24" library="rcl" package="R0805" value="10K" x="28.448" y="70.358" smashed="yes" rot="MR0">
 <attribute name="NAME" x="26.289" y="69.596" size="1.27" layer="26" font="vector" ratio="15" rot="MR0"/>
 <attribute name="VALUE" x="29.083" y="67.818" size="1.27" layer="28" rot="MR0"/>
 </element>
-<element name="R25" library="rcl" package="R0805" value="12K" x="28.448" y="72.39" smashed="yes" rot="MR0">
+<element name="R25" library="rcl" package="R0805" value="10K" x="28.448" y="72.39" smashed="yes" rot="MR0">
 <attribute name="NAME" x="26.289" y="71.628" size="1.27" layer="26" font="vector" ratio="15" rot="MR0"/>
 <attribute name="VALUE" x="29.083" y="69.85" size="1.27" layer="28" rot="MR0"/>
 </element>
 <element name="U$1000" library="SparkFun" package="OSHW-LOGO-L" value="OSHW-LOGOL" x="9.398" y="24.638" smashed="yes" rot="MR0"/>
-<element name="R26" library="rcl" package="R0805" value="12K" x="24.13" y="77.47" smashed="yes" rot="MR180">
+<element name="R26" library="rcl" package="R0805" value="10K" x="24.13" y="77.47" smashed="yes" rot="MR180">
 <attribute name="NAME" x="26.289" y="77.978" size="1.27" layer="26" font="vector" ratio="15" rot="MR180"/>
 <attribute name="VALUE" x="23.495" y="80.01" size="1.27" layer="28" rot="MR180"/>
@@
 <attribute name="VALUE" x="16.764" y="81.534" size="1.27" layer="28" rot="MR180"/>
 </element>
-<element name="R27" library="rcl" package="R0805" value="12K" x="24.13" y="75.438" smashed="yes" rot="MR180">
+<element name="R27" library="rcl" package="R0805" value="10K" x="24.13" y="75.438" smashed="yes" rot="MR180">
 <attribute name="NAME" x="26.289" y="75.946" size="1.27" layer="26" font="vector" ratio="15" rot="MR180"/>
 <attribute name="VALUE" x="23.495" y="77.978" size="1.27" layer="28" rot="MR180"/>
